Commit message: update robot core

File: description/robot_core.xacro (robot description, xacro)
@@ -60,8 +60,8 @@
     </visual>
     <collision>
-        <origin xyz="0.15 0 0.075" rpy="0 0 0"/>
-        <geometry>
-            <box size="0.3 0.3 0.15"/>
+       <geometry>
+            <cylinder length="0.04" radius="0.05" />
         </geometry>
+        <material name="blue"/>
     </collision>
     <xacro:inertial_cylinder mass="0.1" length="0.05" radius="0.05">
@@ -87,8 +87,8 @@
     </visual>
     <collision>
-        <origin xyz="0.15 0 0.075" rpy="0 0 0"/>
         <geometry>
-            <box size="0.3 0.3 0.15"/>
+            <cylinder length="0.04" radius="0.05" />
         </geometry>
+        <material name="blue"/>
     </collision>
     <xacro:inertial_cylinder mass="0.1" length="0.05" radius="0.05">
@@ -113,8 +113,8 @@
     </visual>
     <collision>
-        <origin xyz="0.15 0 0.075" rpy="0 0 0"/>
         <geometry>
-            <box size="0.3 0.3 0.15"/>
+            <sphere radius="0.05" />
         </geometry>
+        <material name="black"/>
     </collision>
     <xacro:inertial_sphere mass="0.1" radius="0.05">
